File: kicad/nrf52840.kicad_pcb (KiCad board)
At the start: 2 copper layers, 40 x 60 mm, 24 parts, among them J1 Conn_01x02, J2 Conn_01x04, J3 Conn_01x06, J4 Conn_01x10, SW1 SW_Push, U1 NRF52840_MS88SF2, U2 AMS1117-3.3, U3 LM2902

Commit message: update
Parts:
- J1: footprint Connector_JST:JST_XH_S2B-XH-A_1x02_P2.50mm_Horizontal -> Connector_JST:JST_XH_S2B-XH-A-1_1x02_P2.50mm_Horizontal
- SW1: footprint Button_Switch_SMD:SW_Push_1P1T_NO_CK_KMR2 -> Button_Switch_SMD:SW_SPST_SKQG_WithStem
- moved SW1 1.78 mm to (48.7, 73.0)
- moved C3 1.70 mm to (58.5, 68.8)
- moved R1 1.70 mm to (56.1, 68.8)
- moved J1 1.68 mm to (50.7, 81.2)
Routing:
- net /~RST: track 34.8 -> 38.4 mm
- net VCC: track 13.0 -> 12.3 mm
